Commit message: Added optional offset for gripper angle, since Nimbus and Prentice have different arms...

File: kinova_description/urdf/j2s7s300.xacro (robot description, xacro)
@@ -98,5 +98,6 @@
     <property name="default_base_trans" value="0 0 0" />
     <property name="default_base_rot" value="0 0 0" />
-    <xacro:macro name="j2s7s300" params="base_parent prefix:=j2s7s300 trans:=${default_base_trans} rot:=${default_base_rot}">
+    <xacro:macro name="j2s7s300" params="base_parent prefix:=j2s7s300 trans:=${default_base_trans}
+    rot:=${default_base_rot} gripper_angle_offset:=0">
         <xacro:gazebo_config robot_namespace="${prefix}"/>
         <xacro:kinova_armlink link_name="${prefix}_link_base" link_mesh="${link_base_mesh}" mesh_no="${link_base_mesh_no}"/>
@@ -125,5 +126,5 @@
           <parent link="${prefix}_link_6" />
           <child link = "${prefix}_link_7" />
-          <origin xyz="0 0.06075 0" rpy="${J_PI/2} 0 0" />
+          <origin xyz="0 0.06075 0" rpy="${J_PI/2} $(gripper_angle_offset) ${0}" />
           <axis xyz="0 0 1" />
           <limit effort="600.8" velocity="0.785"/>

Commit message: syntax error fix

File: kinova_description/urdf/j2s7s300.xacro (robot description, xacro)
@@ -126,5 +126,5 @@
           <parent link="${prefix}_link_6" />
           <child link = "${prefix}_link_7" />
-          <origin xyz="0 0.06075 0" rpy="${J_PI/2} $(gripper_angle_offset) ${0}" />
+          <origin xyz="0 0.06075 0" rpy="${J_PI/2} ${gripper_angle_offset} ${0}" />
           <axis xyz="0 0 1" />
           <limit effort="600.8" velocity="0.785"/>
